Commit message: Updated urdf.xacro so it spawns in gazebo

File: pr2_doors_gazebo_demo/urdf/door.urdf.xacro (robot description, xacro)
@@ -149,5 +149,5 @@
     <turnGravityOff>true</turnGravityOff>
   </gazebo>
-  <gazebo reference="door_link">
+  <!-- <gazebo reference="door_link">
     <latchJoint>handle_joint</latchJoint>
     <latchAngle>-1.57</latchAngle>
@@ -156,9 +156,9 @@
     <latchKd>0.0</latchKd>
     <latchFMax>1000.0</latchFMax>
-  </gazebo>
+  </gazebo> -->
   <joint name="door_joint" type="revolute" >
     <origin xyz="0 0 0.05" rpy="0 0 0" />
     <axis xyz="0 0 1" />
-    <limit lower="-${-M_PI}" upper="${M_PI}" effort="1000" velocity="10" />
+    <limit lower="${-M_PI}" upper="${M_PI}" effort="1000" velocity="10" />
     <safety_controller soft_lower_limit="${-M_PI+0.1}" soft_upper_limit="${M_PI-0.1}"
            k_position="100.0" k_velocity="10.0" />
@@ -365,7 +365,7 @@
     <selfCollide>false</selfCollide>
   </gazebo>
-  <gazebo>
-    <!-- gazebo_ros_p3d for position groundtruth -->
-    <controller:gazebo_ros_p3d name="p3d_door_controller" plugin="libgazebo_ros_p3d.so">
+ <!-- <gazebo>
+     gazebo_ros_p3d for position groundtruth -->
+   <!-- <controller:gazebo_ros_p3d name="p3d_door_controller" plugin="libgazebo_ros_p3d.so">
         <alwaysOn>true</alwaysOn>
         <updateRate>100.0</updateRate>
@@ -381,5 +381,5 @@
       <interface:audio name="gazebo_ros_controller_manager_dummy_iface" />
     </controller:gazebo_ros_controller_manager>
-  </gazebo>
+  </gazebo> -->
   <!-- transmission mechanism controls -->
   <transmission type="pr2_mechanism_model/SimpleTransmission" name="door_trans">
